File: keyswitch.brd (EAGLE design)
At the start: 235.4 x 78.3 mm, 45 parts

Commit message: changes
Routing:
- net N$50: vias 1 -> 0
Changed lines of the file:
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@@
 <wire x1="27.46375" y1="-64.4525" x2="25.24125" y2="-62.23" width="0.635" layer="1"/>
 <wire x1="27.46375" y1="-64.4525" x2="48.895" y2="-64.4525" width="0.635" layer="1"/>
-<wire x1="48.895" y1="-64.4525" x2="46.6725" y2="-62.23" width="0.635" layer="16"/>
+<wire x1="48.895" y1="-64.4525" x2="46.6725" y2="-62.23" width="0.635" layer="1"/>
 <wire x1="48.895" y1="-64.4525" x2="82.2325" y2="-64.4525" width="0.635" layer="1"/>
 <wire x1="80.01" y1="-62.23" x2="82.2325" y2="-64.4525" width="0.635" layer="1"/>
@@
 <wire x1="200.66" y1="-31.4325" x2="200.66" y2="-58.26125" width="0.635" layer="1"/>
 <wire x1="200.66" y1="-58.26125" x2="196.69125" y2="-62.23" width="0.635" layer="1"/>
-<via x="48.895" y="-64.4525" extent="1-16" drill="0.6" shape="square"/>
 </signal>
 <signal name="N$35">
